File: ID_EEPROM.kicad_sch (KiCad schematic)
At the start: 2 parts, among them U2 M24C64

Commit message: cleaned up the repo
Other:
- title: MMS3 Stepper Controler -> MMS3_hat_GPIO_board_basic
Changed lines of the file:
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@@
 	(paper "A4")
 	(title_block
-		(title "MMS3 Stepper Controler")
+		(title "MMS3_hat_GPIO_board_basic")
 		(date "2026-02-25")
-		(rev "R0")
+		(rev "A")
 		(comment 1 "Made by Wojciech Szafrański")
 		(comment 2 "Designed in poland")
