File: MMS3_hat_GPIO_board_basic.kicad_sch (KiCad schematic)
At the start: 10 parts

Commit message: cleaned up the repo
Other:
- removed sheet Buck Regulator
- removed sheet Power Connector
- added sheet GPIO_Expander (GPIO_Expander.kicad_sch)
- title: MMS3 Hat template small (Change Me) -> MMS3_hat_GPIO_board_basic
