File: MMS3_hat_GPIO_board_basic.kicad_sch (KiCad schematic)
At the start: 10 parts

Commit message: added routing and gerber
Parts:
- added C3, C4, C5: 10uF, PCM_JLCPCB:C_0603, symbol PCM_JLCPCB-Capacitors:0603,10uF
- added U3: AMS1117, PCM_JLCPCB:SOT-223-3_L6.5-W3.4-P2.30-LS7.0-BR, symbol PCM_JLCPCB-Power:LDO, 3.3V, 1A
Connections:
- net GND: now also C3.2, C4.2, C5.2, U3.1 (GND)
- new net +3V3: C4.1, C5.1, U3.2 (VOUT), U3.4 (VOUT)
- new net +5V: C3.1, U3.3 (VIN)
Other:
- sheet GPIO_Expander ports: added Chainbus{I2C}; removed none

Commit message: added leds and bom. Revison 1.2
Parts:
- H7, H8, H9, PN1: value ~ -> (none)
